Commit message: feat: commit entire workspace changes for obstacle avoidance optimization

File: src/fishbot_description/urdf/fishbot/fishbot.urdf.xacro (robot description, xacro)
@@ -12,5 +12,5 @@
     <!-- 传感器 -->
     <xacro:imu_xacro xyz="0 0 0.02" />
-    <xacro:laser_xacro xyz="0 0 0.10" />
+    <xacro:laser_xacro xyz="0 0 0.06" />
     <xacro:camera_xacro xyz="0.10 0 0.075" />
     <!-- 执行器主动轮+从动轮 -->

File: src/fishbot_description/urdf/fishbot/plugins/gazebo_sensor_plugin.xacro (robot description, xacro)
@@ -114,4 +114,5 @@
             <sensor type="depth" name="camera_sensor">
                 <plugin name="depth_camera" filename="libgazebo_ros_camera.so">
+                    <camera_name>camera</camera_name>
                     <frame_name>camera_optical_link</frame_name>
                 </plugin>

File: src/fishbot_description/urdf/fishbot/sensor/laser.urdf.xacro (robot description, xacro)
@@ -14,5 +14,5 @@
                 <origin xyz="0 0 0" rpy="0 0 0" />
                 <geometry>
-                    <cylinder length="0.10" radius="0.01" />
+                    <cylinder length="0.02" radius="0.01" />
                 </geometry>
                 <material name="black">
@@ -23,5 +23,5 @@
                 <origin xyz="0 0 0" rpy="0 0 0" />
                 <geometry>
-                    <cylinder length="0.10" radius="0.01" />
+                    <cylinder length="0.02" radius="0.01" />
                 </geometry>
                 <material name="black">
@@ -29,5 +29,5 @@
                 </material>
             </collision>
-            <xacro:cylinder_inertia m="0.01" r="0.01" h="0.10" />
+            <xacro:cylinder_inertia m="0.01" r="0.01" h="0.02" />
         </link>
         <joint name="laser_cylinder_joint" type="fixed">
@@ -61,5 +61,5 @@
             <parent link="laser_cylinder_link" />
             <child link="laser_link" />
-            <origin xyz="0 0 0.05" />
+            <origin xyz="0 0 0.01" />
         </joint>
     </xacro:macro>
