Commit message: feat: raise LiDAR mount height and cylinder height by 3cm to prevent self-scanning chassis

File: src/fishbot_description/urdf/fishbot/fishbot.urdf.xacro (robot description, xacro)
@@ -12,5 +12,5 @@
     <!-- 传感器 -->
     <xacro:imu_xacro xyz="-0.125 0 0.02" />
-    <xacro:laser_xacro xyz="0 0 0.11" />
+    <xacro:laser_xacro xyz="0 0 0.125" />
     <xacro:camera_xacro xyz="0.11 0 0.0" />
     <!-- 执行器：两轮驱动 + 单后万向轮 -->

File: src/fishbot_description/urdf/fishbot/sensor/laser.urdf.xacro (robot description, xacro)
@@ -14,5 +14,5 @@
                 <origin xyz="0 0 0" rpy="0 0 0" />
                 <geometry>
-                    <cylinder length="0.02" radius="0.01" />
+                    <cylinder length="0.05" radius="0.01" />
                 </geometry>
                 <material name="black">
@@ -23,5 +23,5 @@
                 <origin xyz="0 0 0" rpy="0 0 0" />
                 <geometry>
-                    <cylinder length="0.02" radius="0.01" />
+                    <cylinder length="0.05" radius="0.01" />
                 </geometry>
                 <material name="black">
@@ -29,5 +29,5 @@
                 </material>
             </collision>
-            <xacro:cylinder_inertia m="0.01" r="0.01" h="0.02" />
+            <xacro:cylinder_inertia m="0.01" r="0.01" h="0.05" />
         </link>
         <joint name="laser_cylinder_joint" type="fixed">
@@ -61,5 +61,5 @@
             <parent link="laser_cylinder_link" />
             <child link="laser_link" />
-            <origin xyz="0 0 0.01" />
+            <origin xyz="0 0 0.025" />
         </joint>
     </xacro:macro>
