Commit message: fix: revert to front driving wheels and rear caster, resize chassis to 0.45x0.30x0.20, and align base_link to axle

File: src/fishbot_description/urdf/fishbot/base.urdf.xacro (robot description, xacro)
@@ -2,5 +2,5 @@
 <robot xmlns:xacro="http://www.ros.org/wiki/xacro">
    <xacro:include filename="$(find fishbot_description)/urdf/fishbot/common_inertia.xacro" />
-    <xacro:macro name="base_xacro" params="length width depth wheel_radius">
+    <xacro:macro name="base_xacro" params="length width depth wheel_radius x_offset">
      <link name="base_footprint" />
         <joint name="base_joint" type="fixed">
@@ -11,5 +11,5 @@
         <link name="base_link">
             <visual>
-                <origin xyz="0 0 0.0" rpy="0 0 0" />
+                <origin xyz="${x_offset} 0 0.0" rpy="0 0 0" />
                 <geometry>
                     <box size="${depth} ${width} ${length}" />
@@ -20,5 +20,5 @@
             </visual>
             <collision>
-                <origin xyz="0 0 0.0" rpy="0 0 0" />
+                <origin xyz="${x_offset} 0 0.0" rpy="0 0 0" />
                 <geometry>
                     <box size="${depth} ${width} ${length}" />
@@ -28,5 +28,11 @@
                 </material>
             </collision>
-            <xacro:box_inertia m="5.0" w="${depth}" h="${width}" d="${length}"/>
+            <inertial>
+                <origin xyz="${x_offset} 0 0.0" rpy="0 0 0" />
+                <mass value="5.0" />
+                <inertia ixx="${(5.0/12.0) * (width*width + length*length)}" ixy="0.0" ixz="0.0"
+                         iyy="${(5.0/12.0) * (depth*depth + length*length)}" iyz="0.0"
+                         izz="${(5.0/12.0) * (depth*depth + width*width)}" />
+            </inertial>
         </link>
     </xacro:macro>

File: src/fishbot_description/urdf/fishbot/fishbot.urdf.xacro (robot description, xacro)
@@ -9,14 +9,13 @@
     <xacro:include filename="$(find fishbot_description)/urdf/fishbot/actuator/wheel.urdf.xacro" />
     <xacro:include filename="$(find fishbot_description)/urdf/fishbot/actuator/caster.urdf.xacro" />
-    <xacro:base_xacro length="0.23" width="0.35" depth="0.56" wheel_radius="0.08" />
+    <xacro:base_xacro length="0.20" width="0.30" depth="0.45" wheel_radius="0.08" x_offset="-0.125" />
     <!-- 传感器 -->
-    <xacro:imu_xacro xyz="0 0 0.02" />
-    <xacro:laser_xacro xyz="0 0 0.115" />
-    <xacro:camera_xacro xyz="0.29 0 0.0" />
-    <!-- 执行器：四轮驱动 -->
-    <xacro:wheel_xacro wheel_name="front_left" xyz="0.20 0.205 -0.114" radius="0.08" length="0.06" />
-    <xacro:wheel_xacro wheel_name="front_right" xyz="0.20 -0.205 -0.114" radius="0.08" length="0.06" />
-    <xacro:wheel_xacro wheel_name="rear_left" xyz="-0.20 0.205 -0.114" radius="0.08" length="0.06" />
-    <xacro:wheel_xacro wheel_name="rear_right" xyz="-0.20 -0.205 -0.114" radius="0.08" length="0.06" />
+    <xacro:imu_xacro xyz="-0.125 0 0.02" />
+    <xacro:laser_xacro xyz="0 0 0.11" />
+    <xacro:camera_xacro xyz="0.11 0 0.0" />
+    <!-- 执行器：两轮驱动 + 单后万向轮 -->
+    <xacro:wheel_xacro wheel_name="left" xyz="0.0 0.18 -0.10" radius="0.08" length="0.06" />
+    <xacro:wheel_xacro wheel_name="right" xyz="0.0 -0.18 -0.10" radius="0.08" length="0.06" />
+    <xacro:caster_xacro caster_name="rear" xyz="-0.30 0.0 -0.163" />
     <!-- Gazebo 插件 -->
     <xacro:include filename="$(find fishbot_description)/urdf/fishbot/plugins/gazebo_control_plugin.xacro" />

File: src/fishbot_description/urdf/fishbot/plugins/gazebo_control_plugin.xacro (robot description, xacro)
@@ -11,11 +11,9 @@
                 <update_rate>30</update_rate>
                 <!-- wheels -->
-                <num_wheel_pairs>2</num_wheel_pairs>
-                <left_joint>front_left_wheel_joint</left_joint>
-                <left_joint>rear_left_wheel_joint</left_joint>
-                <right_joint>front_right_wheel_joint</right_joint>
-                <right_joint>rear_right_wheel_joint</right_joint>
+                <num_wheel_pairs>1</num_wheel_pairs>
+                <left_joint>left_wheel_joint</left_joint>
+                <right_joint>right_wheel_joint</right_joint>
                 <!-- kinematics -->
-                <wheel_separation>0.41</wheel_separation>
+                <wheel_separation>0.36</wheel_separation>
                 <wheel_diameter>0.16</wheel_diameter>
                 <!-- limits -->
