Commit message: feat: upgrade robot to 4-wheel differential drive with square chassis (0.56x0.35x0.23) and update nav2 configurations

File: src/fishbot_description/urdf/fishbot/actuator/wheel.urdf.xacro (robot description, xacro)
@@ -2,10 +2,10 @@
 <robot xmlns:xacro="http://www.ros.org/wiki/xacro">
    <xacro:include filename="$(find fishbot_description)/urdf/fishbot/common_inertia.xacro" />
-    <xacro:macro name="wheel_xacro" params="wheel_name xyz">
+    <xacro:macro name="wheel_xacro" params="wheel_name xyz radius length">
         <link name="${wheel_name}_wheel_link">
             <visual>
                 <origin xyz="0 0 0" rpy="1.57079 0 0" />
                 <geometry>
-                    <cylinder length="0.04" radius="0.032" />
+                    <cylinder length="${length}" radius="${radius}" />
                 </geometry>
                 <material name="black">
@@ -16,5 +16,5 @@
                 <origin xyz="0 0 0" rpy="1.57079 0 0" />
                 <geometry>
-                    <cylinder length="0.04" radius="0.032" />
+                    <cylinder length="${length}" radius="${radius}" />
                 </geometry>
                 <material name="black">
@@ -22,5 +22,5 @@
                 </material>
             </collision>
-            <xacro:cylinder_inertia m="0.1" h="0.04" r="0.032"/>
+            <xacro:cylinder_inertia m="0.5" h="${length}" r="${radius}"/>
         </link>
         <gazebo reference="${wheel_name}_wheel_link">

File: src/fishbot_description/urdf/fishbot/base.urdf.xacro (robot description, xacro)
@@ -2,10 +2,10 @@
 <robot xmlns:xacro="http://www.ros.org/wiki/xacro">
    <xacro:include filename="$(find fishbot_description)/urdf/fishbot/common_inertia.xacro" />
-    <xacro:macro name="base_xacro" params="length radius">
+    <xacro:macro name="base_xacro" params="length width depth wheel_radius">
      <link name="base_footprint" />
         <joint name="base_joint" type="fixed">
             <parent link="base_footprint" />
             <child link="base_link" />
-            <origin xyz="0.0 0.0 ${length/2.0+0.032-0.001}" rpy="0 0 0" />
+            <origin xyz="0.0 0.0 ${length/2.0+wheel_radius-0.001}" rpy="0 0 0" />
         </joint>
         <link name="base_link">
@@ -13,5 +13,5 @@
                 <origin xyz="0 0 0.0" rpy="0 0 0" />
                 <geometry>
-                    <cylinder length="${length}" radius="${length}" />
+                    <box size="${depth} ${width} ${length}" />
                 </geometry>
                 <material name="blue">
@@ -22,5 +22,5 @@
                 <origin xyz="0 0 0.0" rpy="0 0 0" />
                 <geometry>
-                    <cylinder length="${length}" radius="${length}" />
+                    <box size="${depth} ${width} ${length}" />
                 </geometry>
                 <material name="blue">
@@ -28,5 +28,5 @@
                 </material>
             </collision>
-            <xacro:cylinder_inertia m="1.0" r="${radius}" h="${length}"/>
+            <xacro:box_inertia m="5.0" w="${width}" h="${length}" d="${depth}"/>
         </link>
     </xacro:macro>

File: src/fishbot_description/urdf/fishbot/fishbot.urdf.xacro (robot description, xacro)
@@ -9,14 +9,14 @@
     <xacro:include filename="$(find fishbot_description)/urdf/fishbot/actuator/wheel.urdf.xacro" />
     <xacro:include filename="$(find fishbot_description)/urdf/fishbot/actuator/caster.urdf.xacro" />
-    <xacro:base_xacro length="0.12" radius="0.1" />
+    <xacro:base_xacro length="0.23" width="0.35" depth="0.56" wheel_radius="0.08" />
     <!-- 传感器 -->
     <xacro:imu_xacro xyz="0 0 0.02" />
-    <xacro:laser_xacro xyz="0 0 0.06" />
-    <xacro:camera_xacro xyz="0.10 0 0.075" />
-    <!-- 执行器主动轮+从动轮 -->
-    <xacro:wheel_xacro wheel_name="left" xyz="0 0.10 -0.06" />
-    <xacro:wheel_xacro wheel_name="right" xyz="0 -0.10 -0.06" />
-    <xacro:caster_xacro caster_name="front" xyz="0.08 0.0 -0.076" />
-    <xacro:caster_xacro caster_name="back" xyz="-0.08 0.0 -0.076" />
+    <xacro:laser_xacro xyz="0 0 0.115" />
+    <xacro:camera_xacro xyz="0.29 0 0.0" />
+    <!-- 执行器：四轮驱动 -->
+    <xacro:wheel_xacro wheel_name="front_left" xyz="0.20 0.205 -0.114" radius="0.08" length="0.06" />
+    <xacro:wheel_xacro wheel_name="front_right" xyz="0.20 -0.205 -0.114" radius="0.08" length="0.06" />
+    <xacro:wheel_xacro wheel_name="rear_left" xyz="-0.20 0.205 -0.114" radius="0.08" length="0.06" />
+    <xacro:wheel_xacro wheel_name="rear_right" xyz="-0.20 -0.205 -0.114" radius="0.08" length="0.06" />
     <!-- Gazebo 插件 -->
     <xacro:include filename="$(find fishbot_description)/urdf/fishbot/plugins/gazebo_control_plugin.xacro" />

File: src/fishbot_description/urdf/fishbot/plugins/gazebo_control_plugin.xacro (robot description, xacro)
@@ -11,9 +11,12 @@
                 <update_rate>30</update_rate>
                 <!-- wheels -->
-                <left_joint>left_wheel_joint</left_joint>
-                <right_joint>right_wheel_joint</right_joint>
+                <num_wheel_pairs>2</num_wheel_pairs>
+                <left_joint>front_left_wheel_joint</left_joint>
+                <left_joint>rear_left_wheel_joint</left_joint>
+                <right_joint>front_right_wheel_joint</right_joint>
+                <right_joint>rear_right_wheel_joint</right_joint>
                 <!-- kinematics -->
-                <wheel_separation>0.2</wheel_separation>
-                <wheel_diameter>0.064</wheel_diameter>
+                <wheel_separation>0.41</wheel_separation>
+                <wheel_diameter>0.16</wheel_diameter>
                 <!-- limits -->
                 <max_wheel_torque>400</max_wheel_torque>
