Commit message: feat: lower speed limit to 2.0 m/s and increase rear caster wheel radius to 0.08m with adjusted mounting height to match front wheels

File: src/fishbot_description/urdf/fishbot/actuator/caster.urdf.xacro (robot description, xacro)
@@ -7,5 +7,5 @@
                 <origin xyz="0 0 0" rpy="0 0 0" />
                 <geometry>
-                    <sphere radius="0.016" />
+                    <sphere radius="0.08" />
                 </geometry>
                 <material name="black">
@@ -16,5 +16,5 @@
                 <origin xyz="0 0 0" rpy="0 0 0" />
                 <geometry>
-                    <sphere radius="0.016" />
+                    <sphere radius="0.08" />
                 </geometry>
                 <material name="black">
@@ -22,5 +22,5 @@
                 </material>
             </collision>
-            <xacro:sphere_inertia m="0.01" r="0.016" />
+            <xacro:sphere_inertia m="0.05" r="0.08" />
         </link>
         <gazebo reference="${caster_name}_caster_link">

File: src/fishbot_description/urdf/fishbot/fishbot.urdf.xacro (robot description, xacro)
@@ -17,5 +17,5 @@
     <xacro:wheel_xacro wheel_name="left" xyz="0.0 0.18 -0.10" radius="0.08" length="0.06" />
     <xacro:wheel_xacro wheel_name="right" xyz="0.0 -0.18 -0.10" radius="0.08" length="0.06" />
-    <xacro:caster_xacro caster_name="rear" xyz="-0.30 0.0 -0.163" />
+    <xacro:caster_xacro caster_name="rear" xyz="-0.30 0.0 -0.10" />
     <!-- Gazebo 插件 -->
     <xacro:include filename="$(find fishbot_description)/urdf/fishbot/plugins/gazebo_control_plugin.xacro" />

Commit message: feat: restore 3x3 local costmap, reduce DWB sim_time to 0.7s, restore footprint Y to 28.5cm, and resize caster wheel to 3cm

File: src/fishbot_description/urdf/fishbot/actuator/caster.urdf.xacro (robot description, xacro)
@@ -7,5 +7,5 @@
                 <origin xyz="0 0 0" rpy="0 0 0" />
                 <geometry>
-                    <sphere radius="0.08" />
+                    <sphere radius="0.03" />
                 </geometry>
                 <material name="black">
@@ -16,5 +16,5 @@
                 <origin xyz="0 0 0" rpy="0 0 0" />
                 <geometry>
-                    <sphere radius="0.08" />
+                    <sphere radius="0.03" />
                 </geometry>
                 <material name="black">
@@ -22,5 +22,5 @@
                 </material>
             </collision>
-            <xacro:sphere_inertia m="0.05" r="0.08" />
+            <xacro:sphere_inertia m="0.02" r="0.03" />
         </link>
         <gazebo reference="${caster_name}_caster_link">

File: src/fishbot_description/urdf/fishbot/fishbot.urdf.xacro (robot description, xacro)
@@ -17,5 +17,5 @@
     <xacro:wheel_xacro wheel_name="left" xyz="0.0 0.18 -0.10" radius="0.08" length="0.06" />
     <xacro:wheel_xacro wheel_name="right" xyz="0.0 -0.18 -0.10" radius="0.08" length="0.06" />
-    <xacro:caster_xacro caster_name="rear" xyz="-0.30 0.0 -0.10" />
+    <xacro:caster_xacro caster_name="rear" xyz="-0.30 0.0 -0.15" />
     <!-- Gazebo 插件 -->
     <xacro:include filename="$(find fishbot_description)/urdf/fishbot/plugins/gazebo_control_plugin.xacro" />
