Commit message: refactor: rename packages and files (bot->gazebo, bot_nav2->nav2, fishbot_description->bot_description) to remove all fish references and optimize comments

File: src/bot_description/urdf/bot/actuator/caster.urdf.xacro (robot description, xacro)
@@ -1,5 +1,5 @@
 <?xml version="1.0"?>
 <robot xmlns:xacro="http://www.ros.org/wiki/xacro">
-   <xacro:include filename="$(find fishbot_description)/urdf/fishbot/common_inertia.xacro" />
+   <xacro:include filename="$(find bot_description)/urdf/bot/common_inertia.xacro" />
     <xacro:macro name="caster_xacro" params="caster_name xyz">
         <link name="${caster_name}_caster_link">

File: src/bot_description/urdf/bot/actuator/wheel.urdf.xacro (robot description, xacro)
@@ -1,5 +1,5 @@
 <?xml version="1.0"?>
 <robot xmlns:xacro="http://www.ros.org/wiki/xacro">
-   <xacro:include filename="$(find fishbot_description)/urdf/fishbot/common_inertia.xacro" />
+   <xacro:include filename="$(find bot_description)/urdf/bot/common_inertia.xacro" />
     <xacro:macro name="wheel_xacro" params="wheel_name xyz radius length">
         <link name="${wheel_name}_wheel_link">

File: src/bot_description/urdf/bot/base.urdf.xacro (robot description, xacro)
@@ -1,5 +1,5 @@
 <?xml version="1.0"?>
 <robot xmlns:xacro="http://www.ros.org/wiki/xacro">
-   <xacro:include filename="$(find fishbot_description)/urdf/fishbot/common_inertia.xacro" />
+   <xacro:include filename="$(find bot_description)/urdf/bot/common_inertia.xacro" />
     <xacro:macro name="base_xacro" params="length width depth wheel_radius x_offset">
      <link name="base_footprint" />

File: src/bot_description/urdf/bot/bot.ros2_control.xacro (robot description, xacro)
@@ -1,6 +1,6 @@
 <?xml version="1.0"?>
 <robot xmlns:xacro="http://www.ros.org/wiki/xacro">
-    <xacro:macro name="fishbot_ros2_control">
-    <ros2_control name="FishBotGazeboSystem" type="system">
+    <xacro:macro name="bot_ros2_control">
+        <ros2_control name="BotGazeboSystem" type="system">
             <hardware>
                 <plugin>gazebo_ros2_control/GazeboSystem</plugin>
@@ -34,12 +34,12 @@
         </ros2_control>
         <gazebo>
-        <plugin filename="libgazebo_ros2_control.so" name="gazebo_ros2_control">
-            <parameters>$(find fishbot_description)/config/fishbot_ros2_controller.yaml</parameters>
-            <ros>
-                <remapping>/fishbot_diff_drive_controller/cmd_vel_unstamped:=/cmd_vel</remapping>
-                <remapping>/fishbot_diff_drive_controller/odom:=/odom</remapping>
-            </ros>
-        </plugin>
-</gazebo>
+            <plugin filename="libgazebo_ros2_control.so" name="gazebo_ros2_control">
+                <parameters>$(find bot_description)/config/bot_ros2_controller.yaml</parameters>
+                <ros>
+                    <remapping>/bot_diff_drive_controller/cmd_vel_unstamped:=/cmd_vel</remapping>
+                    <remapping>/bot_diff_drive_controller/odom:=/odom</remapping>
+                </ros>
+            </plugin>
+        </gazebo>
     </xacro:macro>
 </robot>

File: src/bot_description/urdf/bot/sensor/camera.urdf.xacro (robot description, xacro)
@@ -1,5 +1,5 @@
 <?xml version="1.0"?>
 <robot xmlns:xacro="http://www.ros.org/wiki/xacro">
-   <xacro:include filename="$(find fishbot_description)/urdf/fishbot/common_inertia.xacro" />
+   <xacro:include filename="$(find bot_description)/urdf/bot/common_inertia.xacro" />
     <xacro:macro name="camera_xacro" params="xyz">
         <!-- ============相机模块================ -->

File: src/bot_description/urdf/bot/sensor/imu.urdf.xacro (robot description, xacro)
@@ -1,5 +1,5 @@
 <?xml version="1.0"?>
 <robot xmlns:xacro="http://www.ros.org/wiki/xacro">
-   <xacro:include filename="$(find fishbot_description)/urdf/fishbot/common_inertia.xacro" />
+   <xacro:include filename="$(find bot_description)/urdf/bot/common_inertia.xacro" />
     <xacro:macro name="imu_xacro" params="xyz">
         <link name="imu_link">

File: src/bot_description/urdf/bot/sensor/laser.urdf.xacro (robot description, xacro)
@@ -1,5 +1,5 @@
 <?xml version="1.0"?>
 <robot xmlns:xacro="http://www.ros.org/wiki/xacro">
-   <xacro:include filename="$(find fishbot_description)/urdf/fishbot/common_inertia.xacro" />
+   <xacro:include filename="$(find bot_description)/urdf/bot/common_inertia.xacro" />
     <xacro:macro name="laser_xacro" params="xyz">
         <gazebo reference="laser_cylinder_link">
